Commit message: Added apriltag model in husky urdf xacro.

File: Dissertation/simulation/xacro/husky.urdf.xacro (robot description, xacro)
@@ -54,4 +54,5 @@
   <xacro:arg name="robot_namespace" default="$(optenv ROBOT_NAMESPACE /)" />
   <xacro:arg name="tf_prefix" default="$(arg robot_namespace)_tf" />
+  <xacro:arg name="id_cont" default="0"/>
   <xacro:arg name="urdf_extras" default="$(optenv HUSKY_URDF_EXTRAS empty.urdf)" />
   <xacro:arg name="cpr_urdf_extras" default="$(optenv CPR_URDF_EXTRAS empty.urdf)" />
@@ -202,4 +203,26 @@
     <xacro:intel_realsense_mount prefix="camera" topic="realsense" parent_link="realsense_mountpoint"/>
   </xacro:if>
+  <joint name="tag_joint" type="fixed">
+    <origin xyz="0 0 -0.2" rpy="$(arg realsense_rpy)" />
+    <parent link="$(arg realsense_mount)"/>
+    <child link="tag_link" />
+  </joint>
+  <link name="tag_link">
+    <visual>
+      <origin xyz="0 0 0" rpy="0 0 0"/>
+      <geometry>
+        <box size="0.01 0.32 0.32"/>
+      </geometry>
+      <material name="tag_3611_0000$(arg id_cont)"/>
+        <!-- <script>
+          <uri>file:/home/phi/alleff_ws/src/Mestrado/Dissertation/simulation/xacro/tag.material</uri>
+          <name>tag_3611_00000</name>
+        </script>
+      </material> -->
+    </visual>
+  </link>
+  <gazebo reference="tag_link">
+    <material>tag_3611_0000$(arg id_cont)</material>
+  </gazebo>
   <!--
     Add the 3d laser to the sensor arch if needed

Commit message: Changed robot physics. Need to make test.

File: Dissertation/simulation/xacro/husky.urdf.xacro (robot description, xacro)
@@ -59,5 +59,5 @@
   <!-- Included URDF/XACRO Files -->
   <xacro:include filename="$(find husky_description)/urdf/decorations.urdf.xacro" />
-  <xacro:include filename="$(find husky_description)/urdf/wheel.urdf.xacro" />
+  <xacro:include filename="$(find dissertation_simulation)/xacro/wheel.urdf.xacro" />
   <xacro:include filename="$(find dissertation_simulation)/xacro/intel_realsense.urdf.xacro"/>
   <xacro:include filename="$(find husky_description)/urdf/accessories/hokuyo_ust10.urdf.xacro" />
@@ -114,5 +114,5 @@
     <inertial>
       <mass value="46.034" />
-      <origin xyz="-0.00065 -0.085 0.062" />
+      <origin xyz="-0.080 0.000 0.062" />
       <inertia ixx="0.6022" ixy="-0.02364" ixz="-0.1197" iyy="1.7386" iyz="-0.001544" izz="2.0296" />
     </inertial>
