Commit message: Adjusts in Pioneer model to have a realsense built-in

File: pioneer_p3dx/pioneer_description/urdf/materials.xacro (robot description, xacro)
@@ -16,5 +16,5 @@
 work original in ucs-ros-pkg.
  -->
-<robot>
+<robot name="pioneer">
 	<material name="ChassisRed">
 		<color rgba="0.851 0.0 0.0 1.0"/>
@@ -29,12 +29,6 @@
 		<color rgba="1.0 0.811 0.151 1.0"/>
 	</material>
-	<material name="ChassisRed">
-		<color rgba="0.8 0.0 0.0 1.0"/>
-	</material>
 	<material name="TopBlack">
 		<color rgba="0.038 0.038 0.038 1.0"/>
 	</material>
-	<!-- <material name="black">
-  		<color rgba="0.000 0.000 0.000 1.000"/>
-	</material> -->
 </robot>

File: pioneer_p3dx/pioneer_description/urdf/pioneer3dx.xacro (robot description, xacro)
@@ -16,15 +16,21 @@
 work original in ucs-ros-pkg.
  -->
-<robot name="pioneer"
-	xmlns:xacro="http://ros.org/wiki/xacro">
+<robot name="pioneer" xmlns:xacro="http://ros.org/wiki/xacro">
 	<!-- import all gazebo-customization elements, including gazebo colors -->
+	<xacro:include filename="$(find pioneer_description)/urdf/materials.xacro" />
 	<xacro:include filename="$(find pioneer_description)/urdf/pioneer3dx.gazebo" />
 	<!-- import the pioneer 3dx's wheels -->
 	<xacro:include filename="$(find pioneer_description)/urdf/pioneer3dx_wheel.xacro" />
+	<xacro:include filename="$(find pioneer_description)/urdf/intel_realsense.urdf.xacro"/>
 	<!-- chassis -->
+	<link name="dummy"/>
+	<joint name="dummy_joint" type="fixed">
+		<parent link="dummy"/>
+		<child link="base_link"/>
+	</joint>
 	<link name="base_link">
 		<inertial>
 			<mass value="3.5" />
-			<!--<origin xyz="-0.025 0 -0.223"/> -->
+			<origin xyz="-0.025 0 -0.223"/>
 			<origin xyz="-0.05 0 0" />
 			<inertia ixx="1" ixy="0" ixz="0" iyy="1" iyz="0" izz="1" />
@@ -82,5 +88,5 @@
 				<mesh filename="package://pioneer_description/meshes/swivel.stl" />
 			</geometry>
-			<material name="swivel"></material>
+			<material name="WheelBlack"></material>
 		</visual>
 		<collision>
@@ -112,5 +118,5 @@
 				<mesh filename="package://pioneer_description/meshes/center_hubcap.stl" />
 			</geometry>
-			<material name="swivel"></material>
+			<material name="HubcapYellow"></material>
 		</visual>
 		<collision>
@@ -216,3 +222,27 @@
 		<child link="lms100" />
 	</joint>
+	<!-- REALSENSE -->
+	<link name="r_mount">
+		<visual>
+			<origin xyz="0 0 0" rpy="0 0 0" />
+			<geometry>
+				<box size="0.01 0.01 0.15"/>
+			</geometry>
+		</visual>
+	</link>
+	<joint name="r_mount_joint" type="fixed">
+		<axis xyz="0 1 0"/>
+		<origin xyz="0.12 0.0 0.33" rpy="0 0 0"/>
+		<parent link="base_link"/>
+		<child link="r_mount"/>
+	</joint>
+	<link name="realsense_mountpoint"/>
+	<joint name="realsense_joint" type="fixed">
+		<axis xyz="0 1 0"/>
+		<origin xyz="0.12 0.0 0.4" rpy="0 0 0"/>
+		<parent link="base_link"/>
+		<child link="realsense_mountpoint"/>
+	</joint>
+	<xacro:intel_realsense_mount prefix="camera" topic="realsense" parent_link="realsense_mountpoint"/>
+    <xacro:include filename="$(find pioneer_description)/urdf/_d435.urdf.xacro"/>
 </robot>
